File: matrix.kicad_sch (KiCad schematic)
At the start: 126 parts

Commit message: no commit in between is bad
Parts:
- added MX15b1: ~, lck-parts:mx_2u, symbol MX_Alps_Hybrid:MX-NoLED
- added MX29b1: ~, lck-parts:mx_15u, symbol MX_Alps_Hybrid:MX-NoLED
- added MX42b1, MX43b1: ~, lck-parts:mx_225u, symbol MX_Alps_Hybrid:MX-NoLED
- added MX56b1: ~, lck-parts:mx_275u, symbol MX_Alps_Hybrid:MX-NoLED
- D1: value (none) -> D_Small; footprint (none) -> Diode_SMD:D_SOD-123F
- D10, D11, D12, D13, D14, D15, D16, D17, D18, D19, D2, D20, D21, D22, D23, D24, D25, D26, D27, D28, D29, D3, D30, D31, D32, D33, D34, D35, D36, D37, D38, D39, D4, D40, D41, D42, D43, D44, D45, D46, D47, D48, D49, D5, D50, D51, D52, D53, D54, D55, D56, D57, D58, D59, D6, D60, D61, D62, D63, D7, D8, D9: value (none) -> ~; footprint (none) -> Diode_SMD:D_SOD-123F
- MX1: value (none) -> MX-NoLED; footprint (none) -> lck-parts:mx_1u
- MX10, MX11, MX12, MX13, MX14, MX15, MX17, MX18, MX19, MX2, MX20, MX21, MX22, MX23, MX24, MX25, MX26, MX27, MX28, MX3, MX31, MX32, MX33, MX34, MX35, MX36, MX37, MX38, MX39, MX4, MX40, MX41, MX42, MX44, MX45, MX46, MX47, MX48, MX49, MX5, MX50, MX51, MX52, MX53, MX54, MX56, MX58, MX6, MX62, MX7, MX8, MX9: value (none) -> ~; footprint (none) -> lck-parts:mx_1u
- MX16, MX57, MX59, MX61, MX63: value (none) -> ~; footprint (none) -> lck-parts:mx_15u
- MX29: value (none) -> ~; footprint (none) -> lck-parts:mx_iso
- MX30: value (none) -> ~; footprint (none) -> lck-parts:mx_stepped_caps
- MX43: value (none) -> ~; footprint (none) -> lck-parts:mx_125u
- MX55: value (none) -> ~; footprint (none) -> lck-parts:mx_175u
- MX60: value (none) -> ~; footprint (none) -> lck-parts:mx_7u
Connections:
- net COL1: now also MX43b1.1 (COL)
- net COL12: now also MX61.1 (COL)
- net COL13: now also MX62.1 (COL); no longer MX42.1 (COL), MX61.1 (COL)
- net COL14: now also MX42.1 (COL), MX63.1 (COL), MX42b1.1 (COL), MX56b1.1 (COL); no longer MX29.1 (COL), MX62.1 (COL)
- net COL15: now also MX29.1 (COL), MX15b1.1 (COL), MX29b1.1 (COL); no longer MX63.1 (COL)
- net COL6: no longer MX60.1 (COL)
- net COL8: now also MX60.1 (COL)
- net at D15.2 (A), MX15.2 (ROW): now also MX15b1.2 (ROW)
- net at D42.2 (A), MX42.2 (ROW): now also MX42b1.2 (ROW)
- net at D43.2 (A), MX43.2 (ROW): now also MX43b1.2 (ROW)
- net at D56.2 (A), MX56.2 (ROW): now also MX56b1.2 (ROW)
- net at D29.2 (A), MX29.2 (ROW): now also MX29b1.2 (ROW)
Other:
- moved on the sheet: D29, D42, D60, D61, D62, D63, MX29, MX42, MX60, MX61, MX62, MX63
