File: cod67-iso.kicad_sch (KiCad schematic)
At the start: 20 parts, among them J1 AVR-ISP-6, U1 ATmega32U4-AU, U2 PRTR5V0U2X, Y1 16MHz

Commit message: no commit in between is bad
Parts:
- removed U1: ATmega32U4-AU, Package_QFP:TQFP-44_10x10mm_P0.8mm, symbol MCU_Microchip_ATmega:ATmega32U4-AU
- added R6: 10k, Resistor_SMD:R_0402_1005Metric, symbol Device:R_Small
- added SW1: SW_Push, random-keyboard-parts:SKQG-1155865, symbol Switch:SW_Push
- added U1: ATmega32U4-M, Package_DFN_QFN:QFN-44-1EP_7x7mm_P0.5mm_EP5.2x5.2mm, symbol MCU_Microchip_ATmega:ATmega32U4-M
- C1, C2, C3, C4, C5, C6, C7, C8: footprint Capacitor_SMD:C_0805_2012Metric -> Capacitor_SMD:C_0402_1005Metric
- R1, R2, R3, R4, R5: footprint Resistor_SMD:R_0805_2012Metric -> Resistor_SMD:R_0402_1005Metric
Connections:
- net +5V: now also R6.1, U1.14 (VCC), U1.2 (UVCC), U1.24 (AVCC), U1.34 (VCC), U1.44 (AVCC), U1.7 (VBUS)
- net D+: now also U1.4 (D+)
- net D-: now also U1.3 (D-)
- net GND: now also SW1.1, U1.15 (GND), U1.23 (GND), U1.35 (GND), U1.43 (GND), U1.45 (GND), U1.5 (UGND)
- net MISO: now also U1.11 (PB3)
- net MOSI: now also U1.10 (PB2)
- net RST: now also R6.2, SW1.2, U1.13 (~{RESET})
- net XTAL1: now also U1.17 (XTAL1)
- net XTAL2: now also U1.16 (XTAL2)
- net at R1.2: now also U1.33 (~{HWB}/PE2)
- net at C1.1: now also U1.6 (UCAP)
- net SCLK renamed SCK
- net SCK: now also U1.9 (PB1)
- new net COL1: U1.36 (PF7)
- new net COL10: U1.27 (PD7)
- new net COL11: U1.28 (PB4)
- new net COL12: U1.29 (PB5)
- new net COL13: U1.30 (PB6)
- new net COL14: U1.31 (PC6)
- new net COL15: U1.32 (PC7)
- new net COL2: U1.37 (PF6)
- new net COL3: U1.38 (PF5)
- new net COL4: U1.39 (PF4)
- new net COL5: U1.40 (PF1)
- new net COL6: U1.41 (PF0)
- new net COL7: U1.20 (PD2)
- new net COL8: U1.25 (PD4)
- new net COL9: U1.26 (PD6)
- new net LED: U1.8 (PB0)
- new net ROW1: U1.22 (PD5)
- new net ROW2: U1.19 (PD1)
- new net ROW3: U1.18 (PD0)
- new net ROW4: U1.12 (PB7)
- new net ROW5: U1.21 (PD3)
- no-connect marks 3 -> 4

Commit message: change 0402 footprint to 0805 ones
Parts:
- C1, C2, C3, C4, C5, C6, C7, C8: footprint Capacitor_SMD:C_0402_1005Metric -> (none)
- F1: footprint Fuse:Fuse_1206_3216Metric -> (none)
- R1, R2, R3, R4, R5, R6: footprint Resistor_SMD:R_0402_1005Metric -> (none)
