File: leds.kicad_sch (KiCad schematic)
At the start: 20 parts

Commit message: no commit in between is bad
Parts:
- added C10, C11, C12, C13, C14, C15, C16, C17, C18, C19, C20, C21, C22, C23, C24, C25, C26, C27, C28, C9: 0.1uF, Capacitor_SMD:C_0402_1005Metric, symbol Device:C_Small
- LED1, LED11, LED12, LED13, LED14, LED15, LED18, LED2, LED3, LED4, LED5, LED8: footprint (none) -> LED_SMD:LED_WS2812B_PLCC4_5.0x5.0mm_P3.2mm
- LED10: renamed from LED6; footprint (none) -> LED_SMD:LED_WS2812B_PLCC4_5.0x5.0mm_P3.2mm
- LED16: renamed from LED20; footprint (none) -> LED_SMD:LED_WS2812B_PLCC4_5.0x5.0mm_P3.2mm
- LED17: renamed from LED19; footprint (none) -> LED_SMD:LED_WS2812B_PLCC4_5.0x5.0mm_P3.2mm
- LED19: renamed from LED17; footprint (none) -> LED_SMD:LED_WS2812B_PLCC4_5.0x5.0mm_P3.2mm
- LED20: renamed from LED16; footprint (none) -> LED_SMD:LED_WS2812B_PLCC4_5.0x5.0mm_P3.2mm
- LED6: renamed from LED10; footprint (none) -> LED_SMD:LED_WS2812B_PLCC4_5.0x5.0mm_P3.2mm
- LED7: renamed from LED9; footprint (none) -> LED_SMD:LED_WS2812B_PLCC4_5.0x5.0mm_P3.2mm
- LED9: renamed from LED7; footprint (none) -> LED_SMD:LED_WS2812B_PLCC4_5.0x5.0mm_P3.2mm
Connections:
- net +5V: now reaches LED1.1 (VDD), LED10.1 (VDD), LED11.1 (VDD), LED12.1 (VDD), LED13.1 (VDD), LED14.1 (VDD), LED15.1 (VDD), LED16.1 (VDD), LED17.1 (VDD), LED18.1 (VDD), LED19.1 (VDD), LED2.1 (VDD), LED20.1 (VDD), LED3.1 (VDD), LED4.1 (VDD), LED5.1 (VDD), LED6.1 (VDD), LED7.1 (VDD), LED8.1 (VDD), LED9.1 (VDD)
- net +5V: now also C10.2, C11.2, C12.2, C13.1, C14.1, C15.1, C16.1, C17.1, C18.1, C19.2, C20.2, C21.2, C22.2, C23.1, C24.1, C25.1, C26.1, C27.1, C28.2, C9.2
- net GND: now reaches LED1.3 (VSS), LED10.3 (VSS), LED11.3 (VSS), LED12.3 (VSS), LED13.3 (VSS), LED14.3 (VSS), LED15.3 (VSS), LED16.3 (VSS), LED17.3 (VSS), LED18.3 (VSS), LED19.3 (VSS), LED2.3 (VSS), LED20.3 (VSS), LED3.3 (VSS), LED4.3 (VSS), LED5.3 (VSS), LED6.3 (VSS), LED7.3 (VSS), LED8.3 (VSS), LED9.3 (VSS)
- net GND: now also C10.1, C11.1, C12.1, C13.2, C14.2, C15.2, C16.2, C17.2, C18.2, C19.1, C20.1, C21.1, C22.1, C23.2, C24.2, C25.2, C26.2, C27.2, C28.1, C9.1

Commit message: change 0402 footprint to 0805 ones
Parts:
- C10, C11, C12, C13, C14, C15, C16, C17, C18, C19, C20, C21, C22, C23, C24, C25, C26, C27, C28, C9: footprint Capacitor_SMD:C_0402_1005Metric -> (none)
Changed lines of the file:
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@@
       (effects (font (size 1.27 1.27)) (justify left))
     )
-    (property "Footprint" "Capacitor_SMD:C_0402_1005Metric" (id 2) (at 120.65 95.25 0)
+    (property "Footprint" "" (id 2) (at 120.65 95.25 0)
       (effects (font (size 1.27 1.27)) hide)
     )
@@
       (effects (font (size 1.27 1.27)) (justify left))
     )
-    (property "Footprint" "Capacitor_SMD:C_0402_1005Metric" (id 2) (at 167.64 115.57 0)
+    (property "Footprint" "" (id 2) (at 167.64 115.57 0)
       (effects (font (size 1.27 1.27)) hide)
     )
@@
       (effects (font (size 1.27 1.27)) (justify left))
     )
-    (property "Footprint" "Capacitor_SMD:C_0402_1005Metric" (id 2) (at 120.65 74.93 0)
+    (property "Footprint" "" (id 2) (at 120.65 74.93 0)
       (effects (font (size 1.27 1.27)) hide)
     )
@@
       (effects (font (size 1.27 1.27)) (justify left))
     )
-    (property "Footprint" "Capacitor_SMD:C_0402_1005Metric" (id 2) (at 187.96 64.77 0)
+    (property "Footprint" "" (id 2) (at 187.96 64.77 0)
       (effects (font (size 1.27 1.27)) hide)
     )
@@
       (effects (font (size 1.27 1.27)) (justify left))
     )
-    (property "Footprint" "Capacitor_SMD:C_0402_1005Metric" (id 2) (at 167.64 54.61 0)
+    (property "Footprint" "" (id 2) (at 167.64 54.61 0)
       (effects (font (size 1.27 1.27)) hide)
     )
@@
       (effects (font (size 1.27 1.27)) (justify left))
     )
-    (property "Footprint" "Capacitor_SMD:C_0402_1005Metric" (id 2) (at 120.65 115.57 0)
+    (property "Footprint" "" (id 2) (at 120.65 115.57 0)
       (effects (font (size 1.27 1.27)) hide)
     )
@@
       (effects (font (size 1.27 1.27)) (justify left))
     )
-    (property "Footprint" "Capacitor_SMD:C_0402_1005Metric" (id 2) (at 95.25 95.25 0)
+    (property "Footprint" "" (id 2) (at 95.25 95.25 0)
       (effects (font (size 1.27 1.27)) hide)
     )
@@
       (effects (font (size 1.27 1.27)) (justify left))
     )
-    (property "Footprint" "Capacitor_SMD:C_0402_1005Metric" (id 2) (at 144.78 74.93 0)
+    (property "Footprint" "" (id 2) (at 144.78 74.93 0)
       (effects (font (size 1.27 1.27)) hide)
     )
@@
       (effects (font (size 1.27 1.27)) (justify left))
     )
-    (property "Footprint" "Capacitor_SMD:C_0402_1005Metric" (id 2) (at 95.25 74.93 0)
+    (property "Footprint" "" (id 2) (at 95.25 74.93 0)
       (effects (font (size 1.27 1.27)) hide)
     )
@@
       (effects (font (size 1.27 1.27)) (justify left))
     )
-    (property "Footprint" "Capacitor_SMD:C_0402_1005Metric" (id 2) (at 167.64 74.93 0)
+    (property "Footprint" "" (id 2) (at 167.64 74.93 0)
       (effects (font (size 1.27 1.27)) hide)
     )
@@
       (effects (font (size 1.27 1.27)) (justify left))
     )
-    (property "Footprint" "Capacitor_SMD:C_0402_1005Metric" (id 2) (at 187.96 105.41 0)
+    (property "Footprint" "" (id 2) (at 187.96 105.41 0)
       (effects (font (size 1.27 1.27)) hide)
     )
@@
       (effects (font (size 1.27 1.27)) (justify left))
     )
-    (property "Footprint" "Capacitor_SMD:C_0402_1005Metric" (id 2) (at 167.64 95.25 0)
+    (property "Footprint" "" (id 2) (at 167.64 95.25 0)
       (effects (font (size 1.27 1.27)) hide)
     )
@@
       (effects (font (size 1.27 1.27)) (justify left))
     )
-    (property "Footprint" "Capacitor_SMD:C_0402_1005Metric" (id 2) (at 73.66 54.61 0)
+    (property "Footprint" "" (id 2) (at 73.66 54.61 0)
       (effects (font (size 1.27 1.27)) hide)
     )
@@
       (effects (font (size 1.27 1.27)) (justify left))
     )
-    (property "Footprint" "Capacitor_SMD:C_0402_1005Metric" (id 2) (at 76.2 85.09 0)
+    (property "Footprint" "" (id 2) (at 76.2 85.09 0)
       (effects (font (size 1.27 1.27)) hide)
     )
@@
       (effects (font (size 1.27 1.27)) (justify left))
     )
-    (property "Footprint" "Capacitor_SMD:C_0402_1005Metric" (id 2) (at 144.78 115.57 0)
+    (property "Footprint" "" (id 2) (at 144.78 115.57 0)
       (effects (font (size 1.27 1.27)) hide)
     )
@@
       (effects (font (size 1.27 1.27)) (justify left))
     )
-    (property "Footprint" "Capacitor_SMD:C_0402_1005Metric" (id 2) (at 144.78 95.25 0)
+    (property "Footprint" "" (id 2) (at 144.78 95.25 0)
       (effects (font (size 1.27 1.27)) hide)
     )
@@
       (effects (font (size 1.27 1.27)) (justify left))
     )
-    (property "Footprint" "Capacitor_SMD:C_0402_1005Metric" (id 2) (at 95.25 115.57 0)
+    (property "Footprint" "" (id 2) (at 95.25 115.57 0)
       (effects (font (size 1.27 1.27)) hide)
     )
@@
       (effects (font (size 1.27 1.27)) (justify left))
     )
-    (property "Footprint" "Capacitor_SMD:C_0402_1005Metric" (id 2) (at 144.78 54.61 0)
+    (property "Footprint" "" (id 2) (at 144.78 54.61 0)
       (effects (font (size 1.27 1.27)) hide)
     )
@@
       (effects (font (size 1.27 1.27)) (justify left))
     )
-    (property "Footprint" "Capacitor_SMD:C_0402_1005Metric" (id 2) (at 95.25 54.61 0)
+    (property "Footprint" "" (id 2) (at 95.25 54.61 0)
       (effects (font (size 1.27 1.27)) hide)
     )
@@
       (effects (font (size 1.27 1.27)) (justify left))
     )
-    (property "Footprint" "Capacitor_SMD:C_0402_1005Metric" (id 2) (at 120.65 54.61 0)
-      (effects (font (size 1.27 1.27)) hide)
-    )
+    (property "Footprint" "" (id 2) (at 120.65 54.61 0)
+      (effects (font (size 1.27 1.27)) hide)
+    )
